File: ProjektMnozarki/ProjektMnozarki.kicad_sch (KiCad schematic)
At the start: 31 parts, among them IC1 SH8KC6TB1, U1 LM2903, U2 ${SIM.PARAMS}, U3 ${SIM.PARAMS}, U4 ${SIM.PARAMS}, U5 TL431DBZ, U6 ${SIM.PARAMS}, U7 ${SIM.PARAMS}, U8 LT3045xDD

Commit message: Add files via upload
Parts:
- U2, U3, U4: value ${SIM.PARAMS} -> RC4580IDR
- U6, U7: value ${SIM.PARAMS} -> LMH6612MA
Changed lines of the file:
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@@
 			)
 		)
-		(property "Value" "${SIM.PARAMS}"
+		(property "Value" "RC4580IDR"
 			(at 175.26 134.0551 0)
 			(show_name no)
@@
 			)
 		)
-		(property "Value" "${SIM.PARAMS}"
+		(property "Value" "LMH6612MA"
 			(at 109.22 92.1451 0)
 			(show_name no)
@@
 			)
 		)
-		(property "Value" "${SIM.PARAMS}"
+		(property "Value" "LMH6612MA"
 			(at 147.32 94.6851 0)
 			(show_name no)
@@
 			)
 		)
-		(property "Value" "${SIM.PARAMS}"
+		(property "Value" "RC4580IDR"
 			(at 260.35 94.6851 0)
 			(show_name no)
@@
 			)
 		)
-		(property "Value" "${SIM.PARAMS}"
+		(property "Value" "RC4580IDR"
 			(at 218.44 136.5951 0)
 			(show_name no)

Commit message: Add files via upload
Parts:
- added C10, C11, C12, C13, C14, C15, C16, C7, C8, C9: 100n, symbol Device:C
Connections:
- net GND: now also C10.2, C11.2, C12.2, C13.2, C14.2, C15.2, C16.2, C7.2, C8.2, C9.2
- net VCC: now also C10.1, C12.1, C14.1, C16.1, C8.1
- net VEE: now also C11.1, C13.1, C15.1, C7.1, C9.1
